Commit message: Switch to dae mesh, remove unnecessary sensors, update tf frames

File: sensor_kit/twizy_sensor_kit_launch/twizy_sensor_kit_description/urdf/sensor_kit.xacro (robot description, xacro)
@@ -20,25 +20,25 @@
     <xacro:property name="calibration" value="${xacro.load_yaml('$(arg config_dir)/sensor_kit_calibration.yaml')}"/>
     <!-- lidar -->
-    <xacro:VLP-16 parent="sensor_kit_base_link" name="velodyne_top" topic="/points_raw" hz="10" samples="220" gpu="$(arg gpu)">
+    <xacro:VLP-16 parent="sensor_kit_base_link" name="velodyne_sensor" topic="/velodyne_points" hz="10" samples="220" gpu="$(arg gpu)">
       <origin
-        xyz="${calibration['sensor_kit_base_link']['velodyne_top_base_link']['x']}
-             ${calibration['sensor_kit_base_link']['velodyne_top_base_link']['y']}
-             ${calibration['sensor_kit_base_link']['velodyne_top_base_link']['z']}"
-        rpy="${calibration['sensor_kit_base_link']['velodyne_top_base_link']['roll']}
-             ${calibration['sensor_kit_base_link']['velodyne_top_base_link']['pitch']}
-             ${calibration['sensor_kit_base_link']['velodyne_top_base_link']['yaw']}"
+        xyz="${calibration['sensor_kit_base_link']['velodyne']['x']}
+             ${calibration['sensor_kit_base_link']['velodyne']['y']}
+             ${calibration['sensor_kit_base_link']['velodyne']['z']}"
+        rpy="${calibration['sensor_kit_base_link']['velodyne']['roll']}
+             ${calibration['sensor_kit_base_link']['velodyne']['pitch']}
+             ${calibration['sensor_kit_base_link']['velodyne']['yaw']}"
       />
     </xacro:VLP-16>
     <!-- camera, Logitech C920-->
     <xacro:monocular_camera_macro
-      name="camera0/camera"
+      name="default_cam_sensor"
       parent="sensor_kit_base_link"
       namespace=""
-      x="${calibration['sensor_kit_base_link']['camera0/camera_link']['x']}"
-      y="${calibration['sensor_kit_base_link']['camera0/camera_link']['y']}"
-      z="${calibration['sensor_kit_base_link']['camera0/camera_link']['z']}"
-      roll="${calibration['sensor_kit_base_link']['camera0/camera_link']['roll']}"
-      pitch="${calibration['sensor_kit_base_link']['camera0/camera_link']['pitch']}"
-      yaw="${calibration['sensor_kit_base_link']['camera0/camera_link']['yaw']}"
+      x="${calibration['sensor_kit_base_link']['default_cam']['x']}"
+      y="${calibration['sensor_kit_base_link']['default_cam']['y']}"
+      z="${calibration['sensor_kit_base_link']['default_cam']['z']}"
+      roll="${calibration['sensor_kit_base_link']['default_cam']['roll']}"
+      pitch="${calibration['sensor_kit_base_link']['default_cam']['pitch']}"
+      yaw="${calibration['sensor_kit_base_link']['default_cam']['yaw']}"
       fps="30"
       width="1280"
@@ -46,17 +46,4 @@
       fov="1.361"
     />
-    <!-- imu -->
-    <xacro:imu_macro
-      name="sd_imu/imu"
-      parent="sensor_kit_base_link"
-      namespace=""
-      x="${calibration['sensor_kit_base_link']['sd_imu/imu_link']['x']}"
-      y="${calibration['sensor_kit_base_link']['sd_imu/imu_link']['y']}"
-      z="${calibration['sensor_kit_base_link']['sd_imu/imu_link']['z']}"
-      roll="${calibration['sensor_kit_base_link']['sd_imu/imu_link']['roll']}"
-      pitch="${calibration['sensor_kit_base_link']['sd_imu/imu_link']['pitch']}"
-      yaw="${calibration['sensor_kit_base_link']['sd_imu/imu_link']['yaw']}"
-      fps="100"
-    />
   </xacro:macro>
 </robot>

File: vehicle/twizy_vehicle_launch/twizy_vehicle_description/urdf/vehicle.xacro (robot description, xacro)
@@ -1,60 +1,14 @@
 <?xml version="1.0"?>
-<!--
-Copyright (c) 2020 StreetDrone Limited
-Author:  Efimia Panagiotaki
-All rights reserved
--->
-<robot name="sd_twizy" xmlns:xacro="http://www.ros.org/wiki/xacro">
-  <!-- ***************** -->
-  <!-- Imported elements -->
-  <!-- ***************** -->
-  <xacro:include filename="$(find twizy_vehicle_description)/urdf/bases/sd_twizy_body.urdf.xacro" />
-  <xacro:include filename="$(find twizy_vehicle_description)/urdf/wheels/sd_twizy_suspension.urdf.xacro" />
-  <!-- Skipping sensors and using autowares because position updates with sensor_kit calibration files -->
-  <!-- *************** -->
-  <!-- Robots Elements -->
-  <!-- *************** -->
-  <xacro:sd_twizy_base name="sd_twizy"/>
-  <xacro:RL_wheel/>
-  <xacro:RR_wheel/>
-  <xacro:FL_wheel/>
-  <xacro:FR_wheel/>
-  <gazebo>
-    <plugin name="sd_control" filename="libSdControlPlugin.so">
-      <chassis>base_link</chassis>
-      <front_left_wheel>front_left_wheel_joint</front_left_wheel>
-      <front_right_wheel>front_right_wheel_joint</front_right_wheel>
-      <front_left_wheel_steering>front_left_steer_joint</front_left_wheel_steering>
-      <front_right_wheel_steering>front_right_steer_joint</front_right_wheel_steering>
-      <back_left_wheel>rear_left_wheel_joint</back_left_wheel>
-      <back_right_wheel>rear_right_wheel_joint</back_right_wheel>
-      <fl_wheel_steering_p_gain>1e4</fl_wheel_steering_p_gain>
-      <fr_wheel_steering_p_gain>1e4</fr_wheel_steering_p_gain>
-      <fl_wheel_steering_i_gain>0</fl_wheel_steering_i_gain>
-      <fr_wheel_steering_i_gain>0</fr_wheel_steering_i_gain>
-      <fl_wheel_steering_d_gain>3e2</fl_wheel_steering_d_gain>
-      <fr_wheel_steering_d_gain>3e2</fr_wheel_steering_d_gain>
-      <max_speed>22</max_speed>
-      <max_torque>250</max_torque>
-      <front_brake_torque>260</front_brake_torque>
-      <back_brake_torque>260</back_brake_torque>
-      <chassis_aero_force_gain>0.63045</chassis_aero_force_gain>
-    </plugin>
-  </gazebo>
-  <gazebo>
-    <plugin name="p3d" filename="libgazebo_ros_p3d.so">
-      <bodyName>base_link</bodyName>
-      <topicName>base_pose_ground_truth</topicName>
-      <frameName>map</frameName>
-      <updateRate>100.0</updateRate>
-    </plugin>
-  </gazebo>
-  <gazebo>
-    <plugin name="joint_state_publisher" filename="libgazebo_ros_joint_state_publisher.so">
-      <robotNamespace>/sd_twizy</robotNamespace>
-      <jointName>front_left_wheel_joint, front_right_wheel_joint, front_left_steer_joint, front_right_steer_joint, rear_left_wheel_joint, rear_right_wheel_joint</jointName>
-      <updateRate>100.0</updateRate>
-      <alwaysOn>true</alwaysOn>
-    </plugin>
-  </gazebo>
+<robot xmlns:xacro="http://ros.org/wiki/xacro">
+  <!-- load parameter -->
+  <xacro:property name="vehicle_info" value="${xacro.load_yaml('$(find twizy_vehicle_description)/config/vehicle_info.param.yaml')}"/>
+  <!-- vehicle body -->
+  <link name="base_link">
+    <visual>
+      <origin xyz="0 0 0" rpy="${pi/2.0} 0 ${pi/2.0}"/>
+      <geometry>
+        <mesh filename="package://twizy_vehicle_description/mesh/twizy.dae" scale="1 1 1"/>
+      </geometry>
+    </visual>
+  </link>
 </robot>

Commit message: Raise Twizy model in vehicle.xacro and refactor sensor launch
- Previously, Twizy's wheels where clipping the map at the center of the wheel, so I have raised the model by the radius of the rear wheel (which is slightly larger than the front wheel), radius data comes from the original twizy model from StreetDrone: https://github.com/streetdrone-home/SD-TwizyModel/blob/master/streetdrone_model/sd_description/urdf/wheels/sd_twizy_suspension.urdf.xacro

File: sensor_kit/twizy_sensor_kit_launch/twizy_sensor_kit_description/urdf/sensor_kit.xacro (robot description, xacro)
@@ -5,5 +5,4 @@
     <!-- <xacro:include filename="$(find vls_description)/urdf/VLS-128.urdf.xacro"/> -->
     <xacro:include filename="$(find camera_description)/urdf/monocular_camera.xacro"/>
-    <xacro:include filename="$(find imu_description)/urdf/imu.xacro"/>
     <xacro:arg name="gpu" default="false"/>
     <xacro:arg name="config_dir" default="$(find twizy_sensor_kit_description)/config"/>

File: vehicle/twizy_vehicle_launch/twizy_vehicle_description/urdf/vehicle.xacro (robot description, xacro)
@@ -6,5 +6,5 @@
   <link name="base_link">
     <visual>
-      <origin xyz="0 0 0" rpy="${pi/2.0} 0 ${pi/2.0}"/>
+      <origin xyz="0 0 0.281" rpy="${pi/2.0} 0 ${pi/2.0}"/>
       <geometry>
         <mesh filename="package://twizy_vehicle_description/mesh/twizy.dae" scale="1 1 1"/>

Commit message: Skip camera setup, upload extrinsic calibration for lidar

File: sensor_kit/twizy_sensor_kit_launch/twizy_sensor_kit_description/urdf/sensor_kit.xacro (robot description, xacro)
@@ -4,5 +4,5 @@
     <xacro:include filename="$(find velodyne_description)/urdf/VLP-16.urdf.xacro"/>
     <!-- <xacro:include filename="$(find vls_description)/urdf/VLS-128.urdf.xacro"/> -->
-    <xacro:include filename="$(find camera_description)/urdf/monocular_camera.xacro"/>
+    <!-- <xacro:include filename="$(find camera_description)/urdf/monocular_camera.xacro"/> -->
     <xacro:arg name="gpu" default="false"/>
     <xacro:arg name="config_dir" default="$(find twizy_sensor_kit_description)/config"/>
@@ -30,5 +30,5 @@
     </xacro:VLP-16>
     <!-- camera, Logitech C920-->
-    <xacro:monocular_camera_macro
+    <!-- <xacro:monocular_camera_macro
       name="default_cam"
       parent="sensor_kit_base_link"
@@ -44,5 +44,5 @@
       height="720"
       fov="1.361"
-    />
+    /> -->
   </xacro:macro>
 </robot>

File: vehicle/twizy_vehicle_launch/twizy_vehicle_description/urdf/vehicle.xacro (robot description, xacro)
@@ -6,5 +6,5 @@
   <link name="base_link">
     <visual>
-      <origin xyz="0 0 0.281" rpy="${pi/2.0} 0 ${pi/2.0}"/>
+      <origin xyz="0 0 0" rpy="${pi/2.0} 0 ${pi/2.0}"/>
       <geometry>
         <mesh filename="package://twizy_vehicle_description/mesh/twizy.dae" scale="1 1 1"/>
